File: pcb/design/power.kicad_sch (KiCad schematic)
At the start: 8 parts, among them J5 12V INPUT + / -, J6 NC KILL SWITCH, U1 SN74LV125AN, U2 SN74LV125AN

Commit message: feat: finalize 3+3 carrier and bare PCB fabrication package
Connections:
- net 12V_FUSED renamed 12V_PREPOL
Other:
- note added: "12V motor rail only. 12mm shared bus; 2mm per-axis feeds; 1oz copper. Thermal evaluation stopped."
- note removed: "12V motor rail only. 12mm / 2oz shared bus; 2mm per-axis feeds; continuous GND planes."

Commit message: chore: update buffer selection, sourcing BOM and repository rules
Select TI SN74HC125N C2890 without layout changes and document the unresolved powered-off EN guarantee.

- Update design metadata, BOMs, assembly planning and EN verification.

- Include the formatted sourcing workbook and purchasing documentation.

- Add the requested commit and push rules.
Parts:
- U1, U2: value SN74LV125AN -> SN74HC125N
Other:
- note added: "U1/U2 SN74HC125N PDIP14, 3.3V, no Ioff. Unused inputs tied; unused outputs NC."
- note removed: "U1/U2 SN74LV125AN PDIP14, 3.3V, Ioff. Unused inputs tied; unused outputs NC."
